Commit message: working URDF

File: combined.urdf (robot description, URDF)
Before this commit: robot hand_with_arm, 34 links, 34 joints
Links:
- added link base_link_hand, mass 0.0405673074248041; collision mesh filename=package://Assem_w_tip_w_wrist/meshes/base_link_hand.STL; visual mesh filename=package://Assem_w_tip_w_wrist/meshes/base_link_hand.STL
- link base_link: mass 0.0405673074248041 -> 0.83419; geometry collision mesh filename=package://aubo_description/meshes/aubo_i5/collision/base_li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; visual mesh filename=package://aubo_description/meshes/aubo_i5/visual/base_link.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
Joints:
- joint Wrist_Flex_Extension: parent base_link -> base_link_hand
- joint connect: child palm_intermediate_link -> base_link_hand; origin xyz=0 0 0.02 rpy=0 0 0 -> xyz=0 0 0 rpy=0 0 0

File: combined.xacro (robot description, xacro)
@@ -11,6 +11,6 @@
   <joint name="connect" type="fixed">
     <parent link="wrist3_Link"/>
-    <child link="palm_intermediate_link"/>
-    <origin xyz="0 0 0.02" rpy="0 0 0"/>
+    <child link="base_link_hand"/>
+    <origin xyz="0 0 0" rpy="0 0 0"/>
   </joint>
 </robot>

File: hand/Krysalis_Assem_w_tip_w_wrist.xacro (robot description, xacro)
@@ -1,5 +1,5 @@
 <?xml version="1.0" encoding="utf-8"?>
 <robot xmlns:xacro = "http://ros.org/wiki/xacro" name="Assem_w_tip_w_wrist">
-  <link name="base_link">
+  <link name="base_link_hand">
     <inertial>
       <origin xyz="0.00288917703400745 7.19298575992736E-08 0.0333943413697345" rpy="0 0 0" />
@@ -10,5 +10,5 @@
       <origin xyz="0 0 0" rpy="0 0 0" />
       <geometry>
-        <mesh filename="package://Assem_w_tip_w_wrist/meshes/base_link.STL" />
+        <mesh filename="package://Assem_w_tip_w_wrist/meshes/base_link_hand.STL" />
       </geometry>
       <material name="">
@@ -19,5 +19,5 @@
       <origin xyz="0 0 0" rpy="0 0 0" />
       <geometry>
-        <mesh filename="package://Assem_w_tip_w_wrist/meshes/base_link.STL" />
+        <mesh filename="package://Assem_w_tip_w_wrist/meshes/base_link_hand.STL" />
       </geometry>
     </collision>
@@ -736,3 +736,3 @@
     <axis xyz="0 0 0" />
   </joint>
-<link name="palm_intermediate_link" /><joint name="Wrist_Flex_Extension" type="revolute"><parent link="base_link" /><child link="palm_intermediate_link" /><origin xyz="0.00633660798242791 0 0.108612" rpy="1.5707963267949 0 1.5707963267949" /><axis xyz="1 0 0" /><limit lower="-0.907" upper="0.907" effort="1" velocity="1" /></joint><joint name="Wrist_RUD" type="revolute"><parent link="palm_intermediate_link" /><child link="Palm" /><origin xyz="0 0 0" rpy="0 0 0" /><axis xyz="0 0 1" /><limit lower="-0.314" upper="0.314" effort="1" velocity="1" /></joint></robot>
+<link name="palm_intermediate_link" /><joint name="Wrist_Flex_Extension" type="revolute"><parent link="base_link_hand" /><child link="palm_intermediate_link" /><origin xyz="0.00633660798242791 0 0.108612" rpy="1.5707963267949 0 1.5707963267949" /><axis xyz="1 0 0" /><limit lower="-0.907" upper="0.907" effort="1" velocity="1" /></joint><joint name="Wrist_RUD" type="revolute"><parent link="palm_intermediate_link" /><child link="Palm" /><origin xyz="0 0 0" rpy="0 0 0" /><axis xyz="0 0 1" /><limit lower="-0.314" upper="0.314" effort="1" velocity="1" /></joint></robot>

Commit message: add

File: combined.urdf (robot description, URDF)
Before this commit: robot hand_with_arm, 35 links, 34 joints
Joints:
- joint world_joint: origin xyz=0 0 0 rpy=0 0 0 -> xyz=0.0 0.0 0.0 rpy=0.0 0.0 0.0

Commit message: added processing script and simulation

File: combined.urdf (robot description, URDF)
Before this commit: robot hand_with_arm, 35 links, 34 joints
Links:
- link I_B_MCP: geometry collision mesh filename=I_B_MCP.STL; visual mesh filename=I_B_MCP.STL
- link I_DIP: geometry collision mesh filename=I_DIP.STL; visual mesh filename=I_DIP.STL
- link I_DIP_Tip: geometry collision mesh filename=I_DIP_Tip.STL; visual mesh filename=I_DIP_Tip.STL
- link I_MCP: geometry collision mesh filename=I_MCP.STL; visual mesh filename=I_MCP.STL
- link I_PIP: geometry collision mesh filename=I_PIP.STL; visual mesh filename=I_PIP.STL
- link M_DIP: geometry collision mesh filename=M_DIP.STL; visual mesh filename=M_DIP.STL
- link M_DIP_Tip: geometry collision mesh filename=M_DIP_Tip.STL; visual mesh filename=M_DIP_Tip.STL
- link M_MCP: geometry collision mesh filename=M_MCP.STL; visual mesh filename=M_MCP.STL
- link M_PIP: geometry collision mesh filename=M_PIP.STL; visual mesh filename=M_PIP.STL
- link P_B_MCP: geometry collision mesh filename=P_B_MCP.STL; visual mesh filename=P_B_MCP.STL
- link P_DIP: geometry collision mesh filename=P_DIP.STL; visual mesh filename=P_DIP.STL
- link P_DIP_Tip: geometry collision mesh filename=P_DIP_Tip.STL; visual mesh filename=P_DIP_Tip.STL
- link P_MCP: geometry collision mesh filename=P_MCP.STL; visual mesh filename=P_MCP.STL
- link P_PIP: geometry collision mesh filename=P_PIP.STL; visual mesh filename=P_PIP.STL
- link Palm: geometry collision mesh filename=Palm.STL; visual mesh filename=Palm.STL
- link R_B_MCP: geometry collision mesh filename=R_B_MCP.STL; visual mesh filename=R_B_MCP.STL
- link R_DIP: geometry collision mesh filename=R_DIP.STL; visual mesh filename=R_DIP.STL
- link R_DIP_Tip: geometry collision mesh filename=R_DIP_Tip.STL; visual mesh filename=R_DIP_Tip.STL
- link R_MCP: geometry collision mesh filename=R_MCP.STL; visual mesh filename=R_MCP.STL
- link R_PIP: geometry collision mesh filename=R_PIP.STL; visual mesh filename=R_PIP.STL
- link T_CMC: geometry collision mesh filename=T_CMC.STL; visual mesh filename=T_CMC.STL
- link T_IP: geometry collision mesh filename=T_IP.STL; visual mesh filename=T_IP.STL
- link T_IP_Tip: geometry collision mesh filename=T_IP_Tip.STL; visual mesh filename=T_IP_Tip.STL
- link T_MCP: geometry collision mesh filename=T_MCP.STL; visual mesh filename=T_MCP.STL
- link T_P_S: geometry collision mesh filename=T_P_S.STL; visual mesh filename=T_P_S.STL
- link base_link: geometry collision mesh filename=base_link.STL; visual mesh filename=base_link.STL
- link base_link_hand: geometry collision mesh filename=base_link_hand.STL; visual mesh filename=base_link_hand.STL
- link foreArm_Link: geometry collision mesh filename=foreArm_Link.STL; visual mesh filename=foreArm_Link.STL
- link shoulder_Link: geometry collision mesh filename=shoulder_Link.STL; visual mesh filename=shoulder_Link.STL
- link upperArm_Link: geometry collision mesh filename=upperArm_Link.STL; visual mesh filename=upperArm_Link.STL
- link wrist1_Link: geometry collision mesh filename=wrist1_Link.STL; visual mesh filename=wrist1_Link.STL
- link wrist2_Link: geometry collision mesh filename=wrist2_Link.STL; visual mesh filename=wrist2_Link.STL
- link wrist3_Link: geometry collision mesh filename=wrist3_Link.STL; visual mesh filename=wrist3_Link.STL
