Commit message: just in case

File: aubo/aubo_i5.urdf (robot description, URDF)
Before this commit: robot aubo_i5, 8 links, 7 joints
Links:
- link base_link: geometry collision mesh filename=base_link.STL; visual mesh filename=base_link.STL
- link foreArm_Link: geometry collision mesh filename=foreArm_Link.STL; visual mesh filename=foreArm_Link.STL
- link shoulder_Link: geometry collision mesh filename=shoulder_Link.STL; visual mesh filename=shoulder_Link.STL
- link upperArm_Link: geometry collision mesh filename=upperArm_Link.STL; visual mesh filename=upperArm_Link.STL
- link wrist1_Link: geometry collision mesh filename=wrist1_Link.STL; visual mesh filename=wrist1_Link.STL
- link wrist2_Link: geometry collision mesh filename=wrist2_Link.STL; visual mesh filename=wrist2_Link.STL
- link wrist3_Link: geometry collision mesh filename=wrist3_Link.STL; visual mesh filename=wrist3_Link.STL
